File: fixed/spice/i_control_sim/i_control_sim.kicad_sch (KiCad schematic)
At the start: 9 parts, among them Q1 MMBT5551L, U1 LMV321

Commit message: Worked on spice simulations.
Parts:
- removed D1: LED_ALT, LED_SMD:LED_0603_1608Metric, symbol basic_led-rescue:LED_ALT-Device
- removed Q1: MMBT5551L, Package_TO_SOT_SMD:SOT-23, symbol Transistor_BJT:MMBT5551L
- removed R1 (x2): 1G, Resistor_SMD:R_0402_1005Metric, symbol Device:R
- added Q2: MMBT3904, Package_TO_SOT_SMD:SOT-23, symbol Transistor_BJT:MMBT3904
- R1: value 100 -> 30
- renumbered D2 to D1
Connections:
- net Vca: now also Q2.2 (E)
- net Vout: now also Q2.1 (B)
- net at U1.5 (V+), V3.1: now also Q2.3 (C)
Other:
- note added: ".tran 500u 15m .option method=gear abstol=1e-12 reltol=0.005"
- note removed: ".tran 10u 100m .option method=gear"
- note removed: "spice analysis mode:"
- moved on the sheet: D1, R1, U1, V1
