File: fixed/spice/i_control_sim_bjt/i_control_sim_bjt.kicad_sch (KiCad schematic)
At the start: 6 parts, among them Q2 MMBT3904, U1 LMV321

Commit message: Added v0p1 R1 of 18mA fixed.
Parts:
- V3: value dc(10) -> dc(5)
Changed lines of the file:
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@@
       (effects (font (size 1.27 1.27)) (justify right))
     )
-    (property "Sim.Params" "is=0.85n rs=3.3 n=8.6" (at 170.18 77.47 0)
+    (property "Sim.Params" "is=1.42n rs=3.3 n=7.3" (at 170.18 77.47 0)
       (effects (font (size 1.27 1.27)) hide)
     )
@@
       (effects (font (size 1.27 1.27)) (justify left))
     )
-    (property "Value" "dc(10)" (at 110.49 36.9542 0)
+    (property "Value" "dc(5)" (at 110.49 36.9542 0)
       (effects (font (size 1.27 1.27)) (justify left))
     )
