File: fixed/spice/led_sim/led_sim.kicad_sch (KiCad schematic)
At the start: 2 parts

Commit message: Worked on spice simulations.
Parts:
- removed D1: D, symbol Simulation_SPICE:D
- added D3: D, symbol Simulation_SPICE:D
Connections:
- net 0: now also D3.1 (K)
- net at V1.1: now also D3.2 (A)
Other:
- note added: ".tran 1u 3.13m .option method=gear"
- note removed: ".tran 10u 25m .option method=gear"
- note removed: "spice analysis mode:"
- moved on the sheet: V1
Changed lines of the file:
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@@
 (kicad_sch (version 20230121) (generator eeschema)
   (paper "A4")
-  (wire (pts (xy 143.256 65.278) (xy 169.418 65.278))
+  (wire (pts (xy 142.24 83.82) (xy 142.24 87.63))
     (stroke (width 0) (type default))
   )
-  (wire (pts (xy 143.256 65.278) (xy 143.256 73.152))
+  (wire (pts (xy 200.66 81.28) (xy 200.66 87.63))
     (stroke (width 0) (type default))
   )
-  (wire (pts (xy 169.418 81.661) (xy 169.418 87.884))
+  (wire (pts (xy 142.24 63.5) (xy 142.24 73.66))
     (stroke (width 0) (type default))
   )
-  (wire (pts (xy 143.256 83.312) (xy 143.256 87.757))
+  (wire (pts (xy 142.24 63.5) (xy 200.66 63.5))
     (stroke (width 0) (type default))
   )
-  (wire (pts (xy 169.418 65.278) (xy 169.418 74.041))
+  (wire (pts (xy 200.66 63.5) (xy 200.66 73.66))
     (stroke (width 0) (type default))
   )
-  (text ".tran 10u 25m \n.option method=gear" (at 43.307 20.193 0)
+  (text ".tran 1u 3.13m \n.option method=gear" (at 142.24 99.06 0)
     (effects (font (size 1.27 1.27)) (justify left bottom))
   )
-  (text "spice analysis mode: " (at 20.066 20.066 0)
-    (effects (font (size 1.27 1.27) (thickness 0.762) bold) (justify left bottom))
-  )
-  (symbol (lib_id "Simulation_SPICE:VPULSE") (at 143.256 78.232 0) (unit 1)
+  (symbol (lib_id "Simulation_SPICE:VPULSE") (at 142.24 78.74 0) (unit 1)
     (in_bom yes) (on_board yes) (dnp no)
-    (property "Reference" "V1" (at 147.066 76.2912 0)
+    (property "Reference" "V1" (at 146.05 76.7992 0)
       (effects (font (size 1.27 1.27)) (justify left))
     )
-    (property "Value" "VPULSE" (at 147.066 78.8312 0)
+    (property "Value" "VPULSE" (at 146.05 79.3392 0)
       (effects (font (size 1.27 1.27)) (justify left))
     )
-    (property "Footprint" "" (at 143.256 78.232 0)
+    (property "Footprint" "" (at 142.24 78.74 0)
       (effects (font (size 1.27 1.27)) hide)
     )
-    (property "Datasheet" "~" (at 143.256 78.232 0)
+    (property "Datasheet" "~" (at 142.24 78.74 0)
       (effects (font (size 1.27 1.27)) hide)
     )
-    (property "Sim.Pins" "1=+ 2=-" (at 143.256 78.232 0)
+    (property "Sim.Pins" "1=+ 2=-" (at 142.24 78.74 0)
       (effects (font (size 1.27 1.27)) hide)
     )
-    (property "Sim.Type" "PULSE" (at 143.256 78.232 0)
+    (property "Sim.Type" "PULSE" (at 142.24 78.74 0)
       (effects (font (size 1.27 1.27)) hide)
     )
-    (property "Sim.Device" "V" (at 143.256 78.232 0)
+    (property "Sim.Device" "V" (at 142.24 78.74 0)
       (effects (font (size 1.27 1.27)) (justify left) hide)
     )
-    (property "Sim.Params" "pulse(0 5 0 50m 50m 10n 100m)" (at 126.365 83.566 0)
+    (property "Sim.Params" "pulse(0 5 0 5m 5m 10n 10m)" (at 125.349 84.074 0)
       (effects (font (size 1.27 1.27)) (justify left))
     )
@@
     )
   )
-  (symbol (lib_id "Simulation_SPICE:D") (at 169.418 77.851 90) (unit 1)
+  (symbol (lib_id "Simulation_SPICE:D") (at 200.66 77.47 90) (unit 1)
     (in_bom yes) (on_board yes) (dnp no) (fields_autoplaced)
-    (property "Reference" "D1" (at 171.45 74.676 90)
+    (property "Reference" "D3" (at 202.692 74.295 90)
       (effects (font (size 1.27 1.27)) (justify right))
     )
-    (property "Value" "D" (at 171.45 77.216 90)
+    (property "Value" "D" (at 202.692 76.835 90)
       (effects (font (size 1.27 1.27)) (justify right))
     )
-    (property "Footprint" "" (at 169.418 77.851 0)
+    (property "Footprint" "" (at 200.66 77.47 0)
       (effects (font (size 1.27 1.27)) hide)
     )
-    (property "Datasheet" "~" (at 169.418 77.851 0)
+    (property "Datasheet" "~" (at 200.66 77.47 0)
       (effects (font (size 1.27 1.27)) hide)
     )
-    (property "Sim.Device" "D" (at 171.45 79.756 90)
+    (property "Sim.Device" "D" (at 202.692 79.375 90)
       (effects (font (size 1.27 1.27)) (justify right))
     )
-    (property "Sim.Pins" "1=K 2=A" (at 171.45 82.296 90)
+    (property "Sim.Pins" "1=K 2=A" (at 202.692 81.915 90)
       (effects (font (size 1.27 1.27)) (justify right))
     )
-    (property "Sim.Params" "rs=3.3 n=3.1" (at 169.418 77.851 0)
+    (property "Sim.Params" "is=1.417n rs=0 n=7.3" (at 200.66 77.47 0)
       (effects (font (size 1.27 1.27)) hide)
     )
@@
       (project "led_sim"
         (path "/f75e9eee-f78e-49d2-89b7-78a7252546d9"
-          (reference "D1") (unit 1)
+          (reference "D3") (unit 1)
         )
       )
     )
   )
-  (symbol (lib_id "Simulation_SPICE:0") (at 169.418 87.884 0) (unit 1)
+  (symbol (lib_id "Simulation_SPICE:0") (at 200.66 87.63 0) (unit 1)
     (in_bom yes) (on_board yes) (dnp no) (fields_autoplaced)
-    (property "Reference" "#GND04" (at 169.418 90.424 0)
+    (property "Reference" "#GND03" (at 200.66 90.17 0)
       (effects (font (size 1.27 1.27)) hide)
     )
-    (property "Value" "0" (at 169.418 86.614 0)
+    (property "Value" "0" (at 200.66 86.36 0)
       (effects (font (size 1.27 1.27)))
     )
-    (property "Footprint" "" (at 169.418 87.884 0)
+    (property "Footprint" "" (at 200.66 87.63 0)
       (effects (font (size 1.27 1.27)) hide)
     )
-    (property "Datasheet" "~" (at 169.418 87.884 0)
+    (property "Datasheet" "~" (at 200.66 87.63 0)
       (effects (font (size 1.27 1.27)) hide)
     )
@@
       (project "led_sim"
         (path "/f75e9eee-f78e-49d2-89b7-78a7252546d9"
-          (reference "#GND04") (unit 1)
+          (reference "#GND03") (unit 1)
         )
       )
     )
   )
-  (symbol (lib_id "Simulation_SPICE:0") (at 143.256 87.757 0) (unit 1)
+  (symbol (lib_id "Simulation_SPICE:0") (at 142.24 87.63 0) (unit 1)
     (in_bom yes) (on_board yes) (dnp no) (fields_autoplaced)
-    (property "Reference" "#GND02" (at 143.256 90.297 0)
+    (property "Reference" "#GND02" (at 142.24 90.17 0)
       (effects (font (size 1.27 1.27)) hide)
     )
-    (property "Value" "0" (at 143.256 86.487 0)
+    (property "Value" "0" (at 142.24 86.36 0)
       (effects (font (size 1.27 1.27)))
     )
-    (property "Footprint" "" (at 143.256 87.757 0)
+    (property "Footprint" "" (at 142.24 87.63 0)
       (effects (font (size 1.27 1.27)) hide)
     )
-    (property "Datasheet" "~" (at 143.256 87.757 0)
+    (property "Datasheet" "~" (at 142.24 87.63 0)
       (effects (font (size 1.27 1.27)) hide)
     )

Commit message: Added v0p1 R1 of 18mA fixed.
Parts:
- added D1: Vf=3.8, symbol Simulation_SPICE:D
- D3: value D -> white LED, Vf=3.1
Connections:
- net 0: now also D1.1 (K); no longer D3.1 (K)
- net at V1.1: now also D1.2 (A); no longer D3.2 (A)
Other:
- note added: ".tran 1u 3.81m .option method=gear"
- note removed: ".tran 1u 3.13m .option method=gear"
- moved on the sheet: D3
Changed lines of the file:
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@@
     (stroke (width 0) (type default))
   )
-  (text ".tran 1u 3.13m \n.option method=gear" (at 142.24 99.06 0)
+  (text ".tran 1u 3.81m \n.option method=gear" (at 142.24 99.06 0)
     (effects (font (size 1.27 1.27)) (justify left bottom))
   )
@@
     )
   )
-  (symbol (lib_id "Simulation_SPICE:D") (at 200.66 77.47 90) (unit 1)
+  (symbol (lib_id "Simulation_SPICE:D") (at 229.997 94.234 90) (unit 1)
     (in_bom yes) (on_board yes) (dnp no) (fields_autoplaced)
-    (property "Reference" "D3" (at 202.692 74.295 90)
+    (property "Reference" "D3" (at 232.537 90.424 90)
       (effects (font (size 1.27 1.27)) (justify right))
     )
-    (property "Value" "D" (at 202.692 76.835 90)
+    (property "Value" "white LED, Vf=3.1" (at 232.537 92.964 90)
       (effects (font (size 1.27 1.27)) (justify right))
     )
-    (property "Footprint" "" (at 200.66 77.47 0)
+    (property "Footprint" "" (at 229.997 94.234 0)
       (effects (font (size 1.27 1.27)) hide)
     )
-    (property "Datasheet" "~" (at 200.66 77.47 0)
+    (property "Datasheet" "~" (at 229.997 94.234 0)
       (effects (font (size 1.27 1.27)) hide)
     )
-    (property "Sim.Device" "D" (at 202.692 79.375 90)
+    (property "Sim.Device" "D" (at 232.537 95.504 90)
       (effects (font (size 1.27 1.27)) (justify right))
     )
-    (property "Sim.Pins" "1=K 2=A" (at 202.692 81.915 90)
+    (property "Sim.Pins" "1=K 2=A" (at 232.537 98.044 90)
       (effects (font (size 1.27 1.27)) (justify right))
     )
-    (property "Sim.Params" "is=1.417n rs=0 n=7.3" (at 200.66 77.47 0)
+    (property "Sim.Params" "is=1.417n rs=0 n=7.3" (at 229.997 94.234 0)
       (effects (font (size 1.27 1.27)) hide)
     )
@@
         )
       )
+    )
+  )
+  (symbol (lib_id "Simulation_SPICE:D") (at 200.66 77.47 90) (unit 1)
+    (in_bom yes) (on_board yes) (dnp no) (fields_autoplaced)
+    (property "Reference" "D1" (at 203.2 73.66 90)
+      (effects (font (size 1.27 1.27)) (justify right))
+    )
+    (property "Value" "Vf=3.8" (at 203.2 76.2 90)
+      (effects (font (size 1.27 1.27)) (justify right))
+    )
+    (property "Footprint" "" (at 200.66 77.47 0)
+      (effects (font (size 1.27 1.27)) hide)
+    )
+    (property "Datasheet" "~" (at 200.66 77.47 0)
+      (effects (font (size 1.27 1.27)) hide)
+    )
+    (property "Sim.Device" "D" (at 203.2 78.74 90)
+      (effects (font (size 1.27 1.27)) (justify right))
+    )
+    (property "Sim.Pins" "1=K 2=A" (at 203.2 81.28 90)
+      (effects (font (size 1.27 1.27)) (justify right))
+    )
+    (property "Sim.Params" "is=0.85n rs=0 n=8.6" (at 200.66 77.47 0)
+      (effects (font (size 1.27 1.27)) hide)
+    )
+    (pin "1")
+    (pin "2")
+    (instances
+      (project "led_sim"
+        (path "/f75e9eee-f78e-49d2-89b7-78a7252546d9"
+          (reference "D1") (unit 1)
+        )
+      )
