File: fixed/white_24mA/white_24mA.kicad_sch (KiCad schematic)
At the start: 14 parts, among them J1 Conn_01x04, J2 Conn_01x04, Q1 MMBT5551L, U1 TPS61222DCK, U2 LMV321

Commit message: Added 24mA fixed, white led board.
Parts:
- D1: footprint LED_D3mm_custom:LED_D3.0mm -> LED_SMD:LED_0603_1608Metric
Other:
- note added: "Notes, I(LED) current calculation I(LED) = Vset/R1 R1=10 so I(LED) = Vset/10 R2=20k and R3=1k => Vset=0.24V So I(LED) ~0.024A or ~24mA. Resistors R1 10 C854481 R2 20k CC93942 R3 1k C144789 Capacitors C1, C2, C4, 10uF ceramic capacitors C315248 C3, 0.1uF ceramic capacitor C3012376 Inductor L1 4.7uF 0603, C114862"
- note removed: "Notes, I(LED) current calculation I(LED) = Vset/R1 R1=10 so I(LED) = Vset/10 R2=20k and R3=1k => Vset=0.24V So I(LED) ~0.024A or ~24mA. Resistors R1 10 C854481 R2 20k C93942 R3 1k C144789 Capacitors C1, C2, C4, 10uF ceramic capacitors C315248 C3, 0.1uF ceramic capacitor C3012376 Inductor L1 4.7uF 0603, C114862"
Changed lines of the file:
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@@
     (effects (font (size 1.27 1.27)) (justify left bottom))
   )
-  (text "Notes, \n\nI(LED) current calculation\nI(LED) = Vset/R1\nR1=10 so I(LED) = Vset/10\nR2=20k and R3=1k => Vset=0.24V\nSo I(LED) ~0.024A or ~24mA. \n\nResistors\nR1 10 C854481\nR2 20k C93942\nR3  1k C144789\n\nCapacitors\nC1, C2, C4, 10uF  ceramic capacitors C315248\nC3, 0.1uF ceramic capacitor  C3012376\n\nInductor\nL1 4.7uF 0603, C114862\n"
+  (text "Notes, \n\nI(LED) current calculation\nI(LED) = Vset/R1\nR1=10 so I(LED) = Vset/10\nR2=20k and R3=1k => Vset=0.24V\nSo I(LED) ~0.024A or ~24mA. \n\nResistors\nR1 10 C854481\nR2 20k CC93942\nR3  1k C144789\n\nCapacitors\nC1, C2, C4, 10uF  ceramic capacitors C315248\nC3, 0.1uF ceramic capacitor  C3012376\n\nInductor\nL1 4.7uF 0603, C114862\n"
     (at 32.766 130.429 0)
     (effects (font (size 1.27 1.27)) (justify left bottom))
@@
     (pin "4")
     (instances
-      (project "radial_24mA"
+      (project "white_24mA"
         (path "/71f5df2a-3457-4c71-8742-5c7d73c5aae8"
           (reference "J1") (unit 1)
@@
     (pin "4")
     (instances
-      (project "radial_24mA"
+      (project "white_24mA"
         (path "/71f5df2a-3457-4c71-8742-5c7d73c5aae8"
           (reference "J2") (unit 1)
@@
       (effects (font (size 1.27 1.27)) (justify right))
     )
-    (property "Footprint" "LED_D3mm_custom:LED_D3.0mm" (at 157.353 63.881 0)
+    (property "Footprint" "LED_SMD:LED_0603_1608Metric" (at 157.353 63.881 0)
       (effects (font (size 1.27 1.27)) hide)
     )
@@
     (pin "2")
     (instances
-      (project "radial_24mA"
+      (project "white_24mA"
         (path "/71f5df2a-3457-4c71-8742-5c7d73c5aae8"
           (reference "D1") (unit 1)
@@
     (pin "2")
     (instances
-      (project "radial_24mA"
+      (project "white_24mA"
         (path "/71f5df2a-3457-4c71-8742-5c7d73c5aae8"
           (reference "R1") (unit 1)
@@
     (pin "1")
     (instances
-      (project "radial_24mA"
+      (project "white_24mA"
         (path "/71f5df2a-3457-4c71-8742-5c7d73c5aae8"
           (reference "#PWR08") (unit 1)
@@
     (pin "1")
     (instances
-      (project "radial_24mA"
+      (project "white_24mA"
         (path "/71f5df2a-3457-4c71-8742-5c7d73c5aae8"
           (reference "#FLG0101") (unit 1)
@@
     (pin "1")
     (instances
-      (project "radial_24mA"
+      (project "white_24mA"
         (path "/71f5df2a-3457-4c71-8742-5c7d73c5aae8"
           (reference "#FLG0102") (unit 1)
@@
     (pin "1")
     (instances
-      (project "radial_24mA"
+      (project "white_24mA"
         (path "/71f5df2a-3457-4c71-8742-5c7d73c5aae8"
           (reference "#PWR0101") (unit 1)
@@
     (pin "2")
     (instances
-      (project "radial_24mA"
+      (project "white_24mA"
         (path "/71f5df2a-3457-4c71-8742-5c7d73c5aae8"
           (reference "C4") (unit 1)
@@
     (pin "2")
     (instances
-      (project "radial_24mA"
+      (project "white_24mA"
         (path "/71f5df2a-3457-4c71-8742-5c7d73c5aae8"
           (reference "C3") (unit 1)
@@
     (pin "1")
     (instances
-      (project "radial_24mA"
+      (project "white_24mA"
         (path "/71f5df2a-3457-4c71-8742-5c7d73c5aae8"
           (reference "#PWR06") (unit 1)
@@
     (pin "1")
     (instances
-      (project "radial_24mA"
+      (project "white_24mA"
         (path "/71f5df2a-3457-4c71-8742-5c7d73c5aae8"
           (reference "#PWR011") (unit 1)
@@
     (pin "1")
     (instances
-      (project "radial_24mA"
+      (project "white_24mA"
         (path "/71f5df2a-3457-4c71-8742-5c7d73c5aae8"
           (reference "#PWR09") (unit 1)
@@
     (pin "1")
     (instances
-      (project "radial_24mA"
+      (project "white_24mA"
         (path "/71f5df2a-3457-4c71-8742-5c7d73c5aae8"
           (reference "#PWR04") (unit 1)
@@
     (pin "6")
     (instances
-      (project "radial_24mA"
+      (project "white_24mA"
         (path "/71f5df2a-3457-4c71-8742-5c7d73c5aae8"
           (reference "U1") (unit 1)
@@
     (pin "2")
     (instances
-      (project "radial_24mA"
+      (project "white_24mA"
         (path "/71f5df2a-3457-4c71-8742-5c7d73c5aae8"
           (reference "C1") (unit 1)
@@
     (pin "1")
     (instances
-      (project "radial_24mA"
+      (project "white_24mA"
         (path "/71f5df2a-3457-4c71-8742-5c7d73c5aae8"
           (reference "#FLG01") (unit 1)
@@
     (pin "1")
     (instances
-      (project "radial_24mA"
+      (project "white_24mA"
         (path "/71f5df2a-3457-4c71-8742-5c7d73c5aae8"
           (reference "#PWR05") (unit 1)
@@
     (pin "1")
     (instances
-      (project "radial_24mA"
+      (project "white_24mA"
         (path "/71f5df2a-3457-4c71-8742-5c7d73c5aae8"
           (reference "#PWR07") (unit 1)
@@
     (pin "2")
     (instances
-      (project "radial_24mA"
+      (project "white_24mA"
         (path "/71f5df2a-3457-4c71-8742-5c7d73c5aae8"
           (reference "C2") (unit 1)
@@
     (pin "1")
     (instances
-      (project "radial_24mA"
+      (project "white_24mA"
         (path "/71f5df2a-3457-4c71-8742-5c7d73c5aae8"
           (reference "#PWR010") (unit 1)
@@
     (pin "2")
     (instances
-      (project "radial_24mA"
+      (project "white_24mA"
         (path "/71f5df2a-3457-4c71-8742-5c7d73c5aae8"
           (reference "R2") (unit 1)
@@
     (pin "4")
     (instances
-      (project "radial_24mA"
+      (project "white_24mA"
         (path "/71f5df2a-3457-4c71-8742-5c7d73c5aae8"
           (reference "U2") (unit 1)
@@
     (pin "3")
     (instances
-      (project "radial_24mA"
+      (project "white_24mA"
         (path "/71f5df2a-3457-4c71-8742-5c7d73c5aae8"
           (reference "Q1") (unit 1)
@@
     (pin "2")
     (instances
-      (project "radial_24mA"
+      (project "white_24mA"
         (path "/71f5df2a-3457-4c71-8742-5c7d73c5aae8"
           (reference "R3") (unit 1)
@@
     (pin "2")
     (instances
-      (project "radial_24mA"
+      (project "white_24mA"
         (path "/71f5df2a-3457-4c71-8742-5c7d73c5aae8"
           (reference "L1") (unit 1)
