File: fixed/5V_regulator/white_24mA/white_24mA.kicad_pcb (KiCad board)
At the start: 2 copper layers, 25.4 x 20 mm, 18 parts, among them J1 Conn_01x04, J2 Conn_01x04, M1 MountingHole_2.5mm_Pad, M2 MountingHole_2.5mm_Pad, M3 MountingHole_2.5mm_Pad, M4 MountingHole_2.5mm_Pad, Q1 MMBT5551L, U1 TPS61222DCK, U2 LMV321

Commit message: Updated pcb.
Parts:
- R2: value 30k -> 20k
Changed lines of the file:
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@@
     (descr "LED SMD 0603 (1608 Metric), square (rectangular) end terminal, IPC_7351 nominal, (Body size source: http://www.tortai-tech.com/upload/download/2011102023233369053.pdf), generated with kicad-footprint-generator")
     (tags "LED")
-    (property "Sheetfile" "white_16mA.kicad_sch")
+    (property "Sheetfile" "white_24mA.kicad_sch")
     (property "Sheetname" "")
     (property "ki_description" "Light emitting diode")
@@
     (descr "JST SH series connector, SM04B-SRSS-TB (http://www.jst-mfg.com/product/pdf/eng/eSH.pdf), generated with kicad-footprint-generator")
     (tags "connector JST SH top entry")
-    (property "Sheetfile" "white_16mA.kicad_sch")
+    (property "Sheetfile" "white_24mA.kicad_sch")
     (property "Sheetname" "")
     (property "ki_description" "Generic connector, single row, 01x04, script generated (kicad-library-utils/schlib/autogen/connector/)")
@@
     (descr "JST SH series connector, SM04B-SRSS-TB (http://www.jst-mfg.com/product/pdf/eng/eSH.pdf), generated with kicad-footprint-generator")
     (tags "connector JST SH top entry")
-    (property "Sheetfile" "white_16mA.kicad_sch")
+    (property "Sheetfile" "white_24mA.kicad_sch")
     (property "Sheetname" "")
     (property "ki_description" "Generic connector, single row, 01x04, script generated (kicad-library-utils/schlib/autogen/connector/)")
@@
     (descr "Resistor SMD 0402 (1005 Metric), square (rectangular) end terminal, IPC_7351 nominal, (Body size source: IPC-SM-782 page 72, https://www.pcb-3d.com/wordpress/wp-content/uploads/ipc-sm-782a_amendment_1_and_2.pdf), generated with kicad-footprint-generator")
     (tags "resistor")
-    (property "Sheetfile" "white_16mA.kicad_sch")
+    (property "Sheetfile" "white_24mA.kicad_sch")
     (property "Sheetname" "")
     (property "ki_description" "Resistor")
@@
     (descr "SOT, 5 Pin (https://www.jedec.org/sites/default/files/docs/Mo-178c.PDF variant AA), generated with kicad-footprint-generator ipc_gullwing_generator.py")
     (tags "SOT TO_SOT_SMD")
-    (property "Sheetfile" "white_16mA.kicad_sch")
+    (property "Sheetfile" "white_24mA.kicad_sch")
     (property "Sheetname" "")
     (property "ki_description" "Low-Voltage Rail-to-Rail Output Operational Amplifiers, SOT-23-5/SC-70-5")
@@
     (descr "Capacitor SMD 0402 (1005 Metric), square (rectangular) end terminal, IPC_7351 nominal, (Body size source: IPC-SM-782 page 76, https://www.pcb-3d.com/wordpress/wp-content/uploads/ipc-sm-782a_amendment_1_and_2.pdf), generated with kicad-footprint-generator")
     (tags "capacitor")
-    (property "Sheetfile" "white_16mA.kicad_sch")
+    (property "Sheetfile" "white_24mA.kicad_sch")
     (property "Sheetname" "")
     (property "ki_description" "Unpolarized capacitor")
@@
     (descr "Resistor SMD 0402 (1005 Metric), square (rectangular) end terminal, IPC_7351 nominal, (Body size source: IPC-SM-782 page 72, https://www.pcb-3d.com/wordpress/wp-content/uploads/ipc-sm-782a_amendment_1_and_2.pdf), generated with kicad-footprint-generator")
     (tags "resistor")
-    (property "Sheetfile" "white_16mA.kicad_sch")
+    (property "Sheetfile" "white_24mA.kicad_sch")
     (property "Sheetname" "")
     (property "ki_description" "Resistor")
@@
     (descr "Inductor SMD 0603 (1608 Metric), square (rectangular) end terminal, IPC_7351 nominal, (Body size source: http://www.tortai-tech.com/upload/download/2011102023233369053.pdf), generated with kicad-footprint-generator")
     (tags "inductor")
-    (property "Sheetfile" "white_16mA.kicad_sch")
+    (property "Sheetfile" "white_24mA.kicad_sch")
     (property "Sheetname" "")
     (property "ki_description" "Inductor")
@@
     (descr "Resistor SMD 0402 (1005 Metric), square (rectangular) end terminal, IPC_7351 nominal, (Body size source: IPC-SM-782 page 72, https://www.pcb-3d.com/wordpress/wp-content/uploads/ipc-sm-782a_amendment_1_and_2.pdf), generated with kicad-footprint-generator")
     (tags "resistor")
-    (property "Sheetfile" "white_16mA.kicad_sch")
+    (property "Sheetfile" "white_24mA.kicad_sch")
     (property "Sheetname" "")
     (property "ki_description" "Resistor")
@@
         (effects (font (size 1 1) (thickness 0.15)))
     )
-    (fp_text value "30k" (at 0 1.17) (layer "F.Fab") hide
+    (fp_text value "20k" (at 0 1.17) (layer "F.Fab") hide
         (effects (font (size 1 1) (thickness 0.15)))
     )
@@
     (descr "Capacitor SMD 0402 (1005 Metric), square (rectangular) end terminal, IPC_7351 nominal, (Body size source: IPC-SM-782 page 76, https://www.pcb-3d.com/wordpress/wp-content/uploads/ipc-sm-782a_amendment_1_and_2.pdf), generated with kicad-footprint-generator")
     (tags "capacitor")
-    (property "Sheetfile" "white_16mA.kicad_sch")
+    (property "Sheetfile" "white_24mA.kicad_sch")
     (property "Sheetname" "")
     (property "ki_description" "Unpolarized capacitor")
@@
     (descr "SOT-363, SC-70-6")
     (tags "SOT-363 SC-70-6")
-    (property "Sheetfile" "white_16mA.kicad_sch")
+    (property "Sheetfile" "white_24mA.kicad_sch")
     (property "Sheetname" "")
     (property "ki_description" "400 mA Step-Up Converter, Fixed 5V Output Voltage, 0.7-5.5V Input Voltage, SC-70")
@@
     (descr "Capacitor SMD 0402 (1005 Metric), square (rectangular) end terminal, IPC_7351 nominal, (Body size source: IPC-SM-782 page 76, https://www.pcb-3d.com/wordpress/wp-content/uploads/ipc-sm-782a_amendment_1_and_2.pdf), generated with kicad-footprint-generator")
     (tags "capacitor")
-    (property "Sheetfile" "white_16mA.kicad_sch")
+    (property "Sheetfile" "white_24mA.kicad_sch")
     (property "Sheetname" "")
     (property "ki_description" "Unpolarized capacitor")
@@
     (descr "SOT, 3 Pin (https://www.jedec.org/system/files/docs/to-236h.pdf variant AB), generated with kicad-footprint-generator ipc_gullwing_generator.py")
     (tags "SOT TO_SOT_SMD")
-    (property "Sheetfile" "white_16mA.kicad_sch")
+    (property "Sheetfile" "white_24mA.kicad_sch")
     (property "Sheetname" "")
     (property "ki_description" "0.6A Ic, 160V Vce, NPN Transistor, SOT-23")
@@
     (descr "Capacitor SMD 0402 (1005 Metric), square (rectangular) end terminal, IPC_7351 nominal, (Body size source: IPC-SM-782 page 76, https://www.pcb-3d.com/wordpress/wp-content/uploads/ipc-sm-782a_amendment_1_and_2.pdf), generated with kicad-footprint-generator")
     (tags "capacitor")
-    (property "Sheetfile" "white_16mA.kicad_sch")
+    (property "Sheetfile" "white_24mA.kicad_sch")
     (property "Sheetname" "")
     (property "ki_description" "Unpolarized capacitor")
