File: fixed/5V_regulator/radial_16mA/radial_16mA.kicad_pcb (KiCad board)
At the start: 2 copper layers, 25.4 x 20 mm, 18 parts, among them J1 Conn_01x04, J2 Conn_01x04, M1 MountingHole_2.5mm_Pad, M2 MountingHole_2.5mm_Pad, M3 MountingHole_2.5mm_Pad, M4 MountingHole_2.5mm_Pad, Q1 MMBT5551L, U1 TPS61222DCK, U2 LMV321

Commit message: Modified silkscreens on fixed, 5V radial designs.
Added white user writable silkscreen area to both fixed, 5V, radial
designs.
Other:
- board text added: "IControl LED V0.1 R3 www.iorodeo.com"
- board text added: "Radial, I=16mA Vin=3.3-5.0V"
- board text removed: "IControl LED V0.1 R2 www.iorodeo.com Radial, I=16mA Vin=3.3-5.0V"
Changed lines of the file:
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@@
       (drillshape 0)
       (scaleselection 1)
-      (outputdirectory "production/ver_0p1_rev_2/gerber/")
+      (outputdirectory "production/ver_0p1_rev_3/gerber/")
     )
   )
@@
     )
   )
+  (gr_rect (start 69.2023 55.5) (end 74.7776 64.5)
+    (stroke (width 0.12) (type solid)) (fill solid) (layer "B.SilkS"))
   (gr_circle (center 62.7 60) (end 65.1 60)
     (stroke (width 0.25) (type solid)) (fill none) (layer "F.SilkS"))
@@
   (gr_line (start 75.4 52.5) (end 75.4 67.5)
     (stroke (width 0.2) (type solid)) (layer "Edge.Cuts"))
-  (gr_text "IControl LED V0.1 R2\nwww.iorodeo.com\n\n\n\nRadial, I=16mA\nVin=3.3-5.0V" (at 62.7 60.01) (layer "B.SilkS")
+  (gr_text "IControl LED \nV0.1 R3\nwww.iorodeo.com\n" (at 62.7 52.5) (layer "B.SilkS")
     (effects (font (size 1 1) (thickness 0.15)) (justify mirror))
   )
+  (gr_text "Radial, I=16mA\nVin=3.3-5.0V\n" (at 62.7 68) (layer "B.SilkS")
+    (effects (font (size 1 1) (thickness 0.15)) (justify mirror))
+  )
